File: ESP07-RGBstrip-AMP/RGBstrip-ESP07-Controller-Amp-V1.2.sch (EAGLE design)
At the start: 25 parts, among them IC1 LM394, J1 SCREW-TERMINAL_2_0.100, J2 SCREW-TERMINAL_2_0.100, T1 TIP122, T2 TIP122, T3 TIP122

Commit message: added new schematic and board for RGB LED controller/amplifier
Parts:
- removed IC1: LM394, SparkFun-PowerIC:V_REG_78XXSINK
- removed JP1: Norm1, SparkFun-Connectors:M02LOCK_LONGPADS
- removed JP5: Prog01, SparkFun-Connectors:M02LOCK_LONGPADS
- removed JP6: Prog02, SparkFun-Connectors:M02LOCK_LONGPADS
- removed SV1: RGB Cutoff, con-lstb:MA03-2
- added LM3940IT: V_REG_LD1117VXX, SparkFun-PowerIC:V_REG_LD1117VXX
- added SW1, SW2, SW3, SW5, SW6, SW7: (no value), special:SW_DIP-1
- JP4: value +12V / G / R / B -> (none)
Connections:
- net RESET renamed N$1
- removed net N$8: ESP8266-07.GPIO14, JP2.4, SV1.4
- removed net N$9 (its old number): ESP8266-07.GPIO12, JP2.3, SV1.6
- new net N$11: R5.1, SW7.1
- new net N$6: R3.1, SW5.1
- net 3.3V: now also LM3940IT.OUT, SW1.2; no longer IC1.OUT, JP1.1
- net BLUE: now also ESP8266-07.GPIO12, JP2.3, SW5.2; no longer R3.1, SV1.5
- net GND: now also LM3940IT.GND, S1.1, SW2.1, SW3.1; no longer IC1.GND, JP5.1, JP6.1, S1.2
- net GREEN: now also ESP8266-07.GPIO16, JP2.5, SW6.2; no longer R4.1, SV1.1
- net N$12: now also SW3.2; no longer JP6.2
- net N$14: no longer JP5.2
- net N$16: now also SW2.2
- net N$5: now also SW1.1; no longer JP1.2
- net N$7: now also R4.1, SW6.1; no longer ESP8266-07.GPIO16, JP2.5, SV1.2
- net RED: now also ESP8266-07.GPIO14, JP2.4, SW7.2; no longer R5.1, SV1.3
- net VCC: now also LM3940IT.IN; no longer IC1.IN
Other:
- note added: "+12V / G / R / B"
- note added: "v1.2"
- note removed: "v1.0"

Commit message: added V1.2 schematic and board which replaces 2pin jumpers with single dip switches
Parts:
- removed LM3940IT: V_REG_LD1117VXX, SparkFun-PowerIC:V_REG_LD1117VXX
- added IC1: 7805TV, linear:7805TV
- JP4: value (none) -> +12V / G / R / B
- R3, R4, R5: device SparkFun-Resistors:RESISTORPTH-1/4W -> adafruit:R-US_0309/V
- SW1: value (none) -> Norm01
- SW2: value (none) -> Prog
- SW3: value (none) -> Norm02
- SW5: value (none) -> Disconnect01
- SW6: value (none) -> Disconnect03
- SW7: value (none) -> Disconnect02
Connections:
- net BLUE renamed N$26
- removed net N$14: ESP8266-07.GPIO0, JP3.5
- removed net N$16: ESP8266-07.GPIO4, JP3.3, SW2.2
- new net N$12: ESP8266-07.GPIO4, JP3.3
- new net N$9: ESP8266-07.GPIO0, JP3.5, SW2.2
- net 3.3V: now also IC1.VO; no longer LM3940IT.OUT
- net GND: now also IC1.GND, S1.2; no longer LM3940IT.GND, S1.1
- net VCC: now also IC1.VI; no longer LM3940IT.IN
Other:
- note removed: "+12V / G / R / B"
